File: hw/testy.kicad_pcb (KiCad board)
At the start: 2 copper layers, 39.5 x 64.7 mm, 65 parts, among them CN1 SM04B-SRSS-TB (LF)(SN), J1 2pin, J2 1.3_tft, J3 2pin, U1 BQ24075RGTR, U2 AP2112K-3.3TRG1, U3 RP2040, U4 W25Q16JVUXIQ, U5 SM03B-SRSS-TB(LF)(SN)(P), U6 LIS2DW12TR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

Commit message: hw files as they were ordered at jlc
Other:
- board text removed: "banana for scale"
Changed lines of the file:
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@@
-	)
-	(gr_rect
-		(start 16.647 46.6762)
-		(end 49.647 156.6762)
-		(stroke
-			(width 0.1)
-			(type solid)
-		)
-		(fill yes)
-		(layer "F.SilkS")
 	)
 	(gr_rect
@@
 		)
 	)
-	(gr_text "banana\nfor\nscale"
-		(at 32.131 46.5582 0)
-		(layer "F.SilkS" knockout)
-		(effects
-			(font
-				(size 1 1)
-				(thickness 0.2)
-				(bold yes)
-			)
-			(justify bottom)
-		)
-	)

Commit message: change 1M pullup to 100k
Parts:
- R11: value 1M -> 100K
Changed lines of the file:
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@@
 			)
 		)
-		(property "Value" "1M"
+		(property "Value" "100K"
 			(at 0 4 0)
 			(layer "F.Fab")
@@
 			)
 		)
-		(property "LCSC Part" "C26083"
+		(property "LCSC Part" "C25803"
 			(at 0 0 180)
 			(unlocked yes)
