File: hw/testy.kicad_sch (KiCad schematic)
At the start: 65 parts, among them CN1 SM04B-SRSS-TB (LF)(SN), J1 2pin, J2 1.3_tft, J3 2pin, U1 BQ24075RGTR, U2 AP2112K-3.3TRG1, U3 RP2040, U4 W25Q16JVUXIQ, U5 SM03B-SRSS-TB(LF)(SN)(P), U6 LIS2DW12TR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

Commit message: hw files as they were ordered at jlc
Other:
- note added: "qwiic connector"
Changed lines of the file:
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@@
+	)
+	(rectangle
+		(start 233.68 48.26)
+		(end 274.32 88.9)
+		(stroke
+			(width 0)
+			(type default)
+		)
+		(fill
+			(type none)
+		)
 	)
 	(rectangle
@@
 				(thickness 0.6)
 				(bold yes)
+			)
+		)
+	)
+	(text "qwiic connector"
+		(exclude_from_sim no)
+		(at 254.762 51.308 0)
+		(effects
+			(font
+				(size 3 3)
+				(thickness 0.6)
+				(bold yes)

Commit message: change 1M pullup to 100k
Parts:
- R11: value 1M -> 100K; LCSC Part C26083 -> C25803
Changed lines of the file:
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@@
 			)
 		)
-		(property "Value" "1M"
+		(property "Value" "100K"
 			(at 163.068 63.246 0)
 			(effects
@@
 			)
 		)
-		(property "LCSC Part" "C26083"
+		(property "LCSC Part" "C25803"
 			(at 173.99 62.23 0)
 			(effects
